File: hw/bsides_badge.sch (KiCad schematic (older format))
At the start: 0 parts

Commit message: hw: consolidated the schematics to 1 page
Parts:
- added BT1: Battery_Cell, Battery_Holders:Keystone_2466_1xAAA, symbol Battery_Cell
- added C1, C16, C17, C18, C19, C20, C21, C22, C23, C24: 1.0uF, Capacitors_SMD:C_0603, symbol C_Small
- added C10, C9: 47pF, Capacitors_SMD:C_0603, symbol C_Small
- added C11: 10uF, Capacitors_SMD:C_0603, symbol C_Small
- added C12, C14, C2, C4, C5: 0.1uF, Capacitors_SMD:C_0603, symbol C_Small
- added C13, C15, C3: 4.7uF, Capacitors_SMD:C_0603, symbol C_Small
- added C6, C8: 22uF, Capacitors_SMD:C_0805, symbol C_Small
- added C7: 22uF, Capacitors_Tantalum_SMD:CP_Tantalum_Case-A_EIA-3216-18_Reflow, symbol CP1_Small
- added D1, D2, D3: B540, Diodes_SMD:D_SOD-123, symbol B120-E3
- added J3: USB_B, Connectors_USB:USB_Micro-B_Molex_47346-0001, symbol USB_B
- added J4: Micro_SD_Card, SeeedOPL-Connector:MICRO-SD9+4P-SMD-16.1X14.5X1.85MM, symbol Micro_SD_Card
- added J5: CONN_01X24, Connectors_Hirose:Hirose_FH12-24S-0.5SH_1x24_P0.5mm_Horizontal, symbol CONN_01X24
- added L1: 10uH, Inductors_SMD:L_Taiyo-Yuden_NR-60xx_HandSoldering, symbol L_Core_Ferrite
- added L2: 470@100MHz, Inductors_SMD:L_0805, symbol Ferrite_Bead_Small
- added L3: 22uH, Inductors_SMD:L_Taiyo-Yuden_NR-40xx_HandSoldering, symbol L_Core_Ferrite
- added Q1: 2N7002, TO_SOT_Packages_SMD:SOT-23, symbol 2N7002
- added Q2: CJ2302, TO_SOT_Packages_SMD:SOT-23, symbol 2N7002
- added R1, R15, R16, R17, R18, R19, R2, R20, R6: 10k, Resistors_SMD:R_0603, symbol R_Small_us
- added R10, R11, R12, R13, R14, R21, R22, R9: 0, Resistors_SMD:R_0603, symbol R_Small_us
- added R23: ??, Resistors_SMD:R_0603, symbol R_Small_us
- added R3: 470, Resistors_SMD:R_0603, symbol R_Small_us
- added R4: 1k, Resistors_SMD:R_0603, symbol R_Small_us
- added R5: 1M, Resistors_SMD:R_0603, symbol R_Small_us
- added R7, R8: 22, Resistors_SMD:R_0603, symbol R_Small_us
- added SW1: SW_Push, Buttons_Switches_SMD:SW_SPST_SKQG, symbol SW_Push
- added TP1, TP10, TP11, TP12, TP13, TP14, TP15, TP2, TP3, TP4, TP5, TP6, TP7, TP8, TP9: TEST_POINT, Wire_Pads:SolderWirePad_single_0-8mmDrill, symbol CONN_01X01
- added U1: ESP32-WROOM, ESP32-footprints-Lib:ESP32-WROOM, symbol ESP32-WROOM
- added U2: ETA1036-33S2F-T, TO_SOT_Packages_SMD:SOT-23-5, symbol PMIC-ETA1036-50S2F-T_SOT23-5_
- added U3: CJT1117-3.3, TO_SOT_Packages_SMD:SOT-223-3_TabPin2, symbol LT1117-3.3
- added U4: FT230XS, Housings_SSOP:SSOP-16_3.9x4.9mm_Pitch0.635mm, symbol FT230XS
Connections:
- new net: J4.1 (DAT2), R20.1, R9.1
- new net: J4.2 (DAT3/CD), R10.1, R19.1
- new net: J4.3 (CMD), R11.1, R18.1
- new net: J4.5 (CLK), R12.1, R17.1
- new net: J4.7 (DAT0), R13.1, R16.1
- new net: J4.8 (DAT1), R14.1, R15.1
- new net: J5.18 (P18), TP12.1 (P1)
- new net: J5.19 (P19), TP11.1 (P1)
- new net: J5.24 (P24), TP10.1 (P1)
- new net: J5.6 (P6), TP13.1 (P1)
- new net: R21.2, U4.1 (TXD)
- new net: TP6.1 (P1), U4.14 (CBUS1)
- new net: TP5.1 (P1), U4.15 (CBUS0)
- new net: TP8.1 (P1), U4.16 (CBUS3)
- new net: TP3.1 (P1), U4.2 (~RTS)
- new net: R22.2, U4.4 (RXD)
- new net: TP4.1 (P1), U4.6 (~CTS)
- new net: TP7.1 (P1), U4.7 (CBUS2)
- new net: R7.1, U4.8 (USBDP)
- new net: R8.1, U4.9 (USBDM)
- new net: C11.1, J3.1 (VBUS), L2.1
- new net: C10.1, J3.2 (D-), R8.2
- new net: C9.1, J3.3 (D+), R7.2
- new net: Q1.3 (D), R5.1, TP1.1 (P1), U2.3 (EN)
- new net: L1.2, U2.5 (SW)
- new net: C2.1, Q1.1 (G), R1.1, R4.2
- new net: R3.1, SW1.2
- new net: C18.1, D2.2 (A), L3.2, Q2.3 (D)
- new net: C18.2, D1.2 (A), D3.1 (K)
- new net +3V3: C1.1, C15.1, C6.1, C7.1, C8.1, J4.4 (VDD), J5.10 (P10), J5.7 (P7), J5.9 (P9), L3.1, R15.2, R16.2, R17.2, R18.2, R19.2, R2.2, R20.2, U1.2 (3V3), U2.1 (OUT), U3.2 (VO)
- new net +5V: C12.1, C13.1, C5.1, L2.2, R1.2, U3.3 (VI), U4.12 (VCC)
- new net 3V3OUT: C14.1, TP2.1 (P1), U4.10 (3V3OUT), U4.11 (~RESET), U4.3 (VCCIO)
- new net DISP_BUSY: J5.16 (P16), U1.33 (IO21)
- new net DISP_CS: J5.13 (P13), U1.30 (IO18)
- new net DISP_D: J5.14 (P14), U1.31 (IO19)
- new net DISP_MOSI: J5.11 (P11), U1.28 (IO17)
- new net DISP_RESETn: J5.15 (P15), U1.37 (IO23)
- new net DISP_SCK: J5.12 (P12), U1.29 (IO5)
- new net EN: C4.1, R2.1, R3.2, U1.3 (EN)
- new net GDR: J5.23 (P23), Q2.1 (G)
- new net GND: BT1.2 (-), C1.2, C10.2, C11.2, C12.2, C13.2, C14.2, C15.2, C16.2, C19.2, C2.2, C20.2, C21.2, C22.2, C23.1, C24.2, C3.2, C4.2, C5.2, C6.2, C7.2, C8.2, C9.2, D1.1 (K), J3.4 (GND), J3.5 (Shield), J4.6 (VSS), J4.9 (SHIELD), J5.17 (P17), J5.8 (P8), Q1.2 (S), R23.1, R4.1, SW1.1, U1.1 (GND), U1.15 (GND), U1.38 (GND), U1.39 (GND-PAD), U2.2 (GND), U3.1 (GND), U4.13 (GND), U4.5 (GND)
- new net PREVGH: C22.1, D2.1 (K), J5.4 (P4), TP14.1 (P1)
- new net PREVGL: C23.2, D3.2 (A), J5.2 (P2), TP15.1 (P1)
- new net RESE: J5.22 (P22), Q2.2 (S), R23.2, TP9.1 (P1)
- new net SD_CLK: R12.2, U1.13 (IO14)
- new net SD_CMD: R11.2, U1.23 (IO15)
- new net SD_DAT0: R13.2, U1.24 (IO2)
- new net SD_DAT1: R14.2, U1.26 (IO4)
- new net SD_DAT2: R9.2, U1.14 (IO12)
- new net SD_DAT3: R10.2, U1.16 (IO13)
- new net UART_RX: R21.1, U1.34 (RXD0)
- new net UART_TX: R22.1, U1.35 (TXD0)
- new net VBATT: BT1.1 (+), C3.1, L1.1, R5.2, R6.2, U2.4 (IN)
- new net VCI: C20.1
- new net VCOM: C16.1, J5.1 (P1)
- new net VGH: C24.1, J5.20 (P20)
- new net VGL: C21.1, J5.21 (P21)
- new net VSH: C19.1, J5.5 (P5)
- new net VSL: C17.1, J5.3 (P3)
Other:
- note added: "BATTERY CONNECTOR"
- note added: "DO WE NEED SD CONNECTOR \nWITH CARD-DETECT?\n"
- note added: "SOT-223"

Commit message: hw: Board partially routed
- Board initially routed
- Started on BOM for system
- Added 0-ohm resistors to SPI lines in e-paper display
-- Need to netlist this still
- Added TODO list in schematic
Parts:
- added R? (x6): 0, Resistors_SMD:R_0603, symbol R_Small_us
- Q1, Q2: symbol 2N7002 -> 2N7002-RESCUE-bsides_badge
Connections:
- net DISP_BUSY: now also R?.2; no longer J5.16 (P16)
- net DISP_CS: now also R?.2; no longer J5.13 (P13)
- net DISP_D: now also R?.2; no longer J5.14 (P14)
- net DISP_MOSI: now also R?.2; no longer J5.11 (P11)
- net DISP_RESETn: now also R?.2; no longer J5.15 (P15)
- net DISP_SCK: now also R?.2; no longer J5.12 (P12)
- new net: J5.11 (P11), R?.1
- new net: J5.12 (P12), R?.1
- new net: J5.13 (P13), R?.1
- new net: J5.14 (P14), R?.1
- new net: J5.15 (P15), R?.1
- new net: J5.16 (P16), R?.1
Other:
- note added: "TODO:\n- ADD LEDS FOR RX/TX\n- ADD CIRCUIT FOR AUTOMATIC PROGRAMMING (IF POSSIBLE)\n- FINISH VBATT SENSE CIRCUIT\n\n"
- moved on the sheet: J4, R10, R11, R12, R13, R14, R15, R16, R17, R18, R19, R20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
