File: hw/bsides_badge.kicad_pcb (KiCad board)
At the start: 2 copper layers, 79 parts, among them J3 USB_B, J4 Micro_SD_Card, J5 CONN_01X24, Q1 2N7002, Q2 CJ2302, SW1 SW_Push, U1 ESP32-WROOM, U2 ETA1036-33S2F-T, U3 CJT1117-3.3, U4 FT230XS

Commit message: hw: Board partially routed
- Board initially routed
- Started on BOM for system
- Added 0-ohm resistors to SPI lines in e-paper display
-- Need to netlist this still
- Added TODO list in schematic
Parts:
- U4: moved to B.Cu
- moved TP9 110.1 mm to (136.5, 46.5)
- moved TP12 103.8 mm to (139.5, 46.5)
- moved TP15 98.3 mm to (148.5, 46.5)
- moved TP10 95.7 mm to (133.5, 46.5)
- moved TP11 90.9 mm to (142.5, 46.5)
- moved TP2 90.4 mm to (111.5, 99.0)
- moved R6 87.3 mm to (101.5, 131.0)
- moved TP13 86.0 mm to (151.5, 46.5)
- moved TP4 85.5 mm to (117.0, 115.0)
- moved TP14 84.6 mm to (145.5, 46.5)
- moved L3 83.1 mm to (157.0, 63.0)
- moved R3 82.5 mm to (102.0, 92.0), turned to 90 degrees
- moved R5 80.4 mm to (104.0, 128.0), turned to 270 degrees
- moved D3 79.1 mm to (156.0, 69.0)
- moved J5 78.5 mm to (142.0, 65.0), turned to 180 degrees
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Routing:
- net GND: track 0.00 -> 112.6 mm
- net +3V3: track 0.00 -> 81.2 mm, vias 0 -> 2
- net /SD_CLK: track 0.00 -> 74.9 mm
- net /SD_DAT2: track 0.00 -> 69.8 mm
- net /SD_DAT3: track 0.00 -> 64.5 mm, vias 0 -> 2
- net /SD_CMD: track 0.00 -> 60.0 mm, vias 0 -> 2
- net /SD_DAT1: track 0.00 -> 56.2 mm, vias 0 -> 2
- net Net-(R22-Pad2): track 0.00 -> 55.7 mm, vias 0 -> 3
- net /SD_DAT0: track 0.00 -> 55.5 mm, vias 0 -> 2
- net Net-(R21-Pad2): track 0.00 -> 47.2 mm, vias 0 -> 3
- net +5V: track 0.00 -> 38.1 mm, vias 0 -> 3
- net /VBATT: track 0.00 -> 34.5 mm
- net /EN: track 0.00 -> 26.8 mm
- net /DISP_MOSI: track 0.00 -> 21.1 mm
- net /DISP_SCK: track 0.00 -> 19.5 mm
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Other:
- board outline added: 100 x 100 mm

Commit message: hw: Completed most of the routing
Parts:
- moved R11 34.1 mm to (134.1, 85.1)
- moved R9 34.1 mm to (134.1, 82.0)
- moved R13 34.1 mm to (134.1, 87.9)
- moved R12 31.4 mm to (136.9, 86.6)
- moved R10 31.4 mm to (136.9, 83.6)
- moved R14 31.3 mm to (136.9, 89.4)
- moved R20 31.1 mm to (140.0, 79.5), turned to 90 degrees
- moved R19 29.3 mm to (141.7, 79.5), turned to 90 degrees
- moved C16 28.3 mm to (154.2, 62.0)
- moved R18 27.5 mm to (143.5, 79.5), turned to 90 degrees
- moved TP14 25.9 mm to (145.5, 72.4)
- moved R17 25.9 mm to (145.3, 79.5), turned to 90 degrees
- moved TP12 25.1 mm to (138.9, 71.6)
- moved C17 25.0 mm to (154.2, 60.5)
- moved TP13 24.7 mm to (144.3, 70.1)
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Routing:
- net +3V3: track 81.2 -> 204.7 mm, vias 2 -> 7
- net Net-(J4-Pad7): track 0.00 -> 62.5 mm, vias 0 -> 2
- net Net-(J4-Pad3): track 0.00 -> 60.4 mm, vias 0 -> 2
- net Net-(J4-Pad8): track 1.50 -> 61.5 mm, vias 0 -> 2
- net Net-(J4-Pad5): track 0.00 -> 58.9 mm, vias 0 -> 2
- net Net-(J4-Pad1): track 0.00 -> 57.0 mm
- net Net-(J4-Pad2): track 0.00 -> 55.9 mm, vias 0 -> 2
- net /SD_DAT0: track 55.5 -> 20.0 mm
- net /SD_CMD: track 60.0 -> 25.4 mm
- net /SD_DAT2: track 69.8 -> 35.5 mm
- net /SD_CLK: track 74.9 -> 42.1 mm
- net /SD_DAT1: track 56.2 -> 23.5 mm
- net /SD_DAT3: track 64.5 -> 33.1 mm
- net /DISP_RESETn: track 0.00 -> 30.5 mm, vias 0 -> 2
- net /DISP_CS: track 0.00 -> 27.0 mm
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